File: Regulador_tension_5V/Regulador_tension_5V.sch (KiCad schematic (older format))
At the start: 10 parts, among them P1 CONN_01X02, P2 CONN_01X02, U1 LM7805

Commit message: Añadimos la versión 1.1 del regulador
Parts:
- P1, P2: footprint Socket_Strips:Socket_Strip_Angled_1x02 -> Connectors_Molex:Connector_Molex_PicoBlade_53047-0210
- R1: footprint Resistors_ThroughHole:Resistor_Ceramic_Horizontal_L19mm-W8mm-H8mm-p25mm -> Resistors_ThroughHole:Resistor_Horizontal_RM15mm
Changed lines of the file:
@@
 LIBS:contrib
 LIBS:valves
+LIBS:Regulador_tension_5V-cache
 EELAYER 25 0
 EELAYER END
@@
 F 0 "P1" H 1450 1740 50  0000 C CNN
 F 1 "CONN_01X02" V 1550 1590 50  0000 C CNN
-F 2 "Socket_Strips:Socket_Strip_Angled_1x02" H 1450 1590 50  0001 C CNN
+F 2 "Connectors_Molex:Connector_Molex_PicoBlade_53047-0210" H 1450 1590 50  0001 C CNN
 F 3 "" H 1450 1590 50  0000 C CNN
 	1    1450 1590
@@
 F 0 "R1" V 5355 1645 50  0000 C CNN
 F 1 "1k" V 5275 1645 50  0000 C CNN
-F 2 "Resistors_ThroughHole:Resistor_Ceramic_Horizontal_L19mm-W8mm-H8mm-p25mm" V 5205 1645 50  0001 C CNN
+F 2 "Resistors_ThroughHole:Resistor_Horizontal_RM15mm" V 5205 1645 50  0001 C CNN
 F 3 "" H 5275 1645 50  0000 C CNN
 	1    5275 1645
@@
 F 0 "P2" H 5980 1720 50  0000 C CNN
 F 1 "CONN_01X02" V 6080 1570 50  0000 C CNN
-F 2 "Socket_Strips:Socket_Strip_Angled_1x02" H 5980 1570 50  0001 C CNN
+F 2 "Connectors_Molex:Connector_Molex_PicoBlade_53047-0210" H 5980 1570 50  0001 C CNN
 F 3 "" H 5980 1570 50  0000 C CNN
 	1    5980 1570
