File: ATtiny85_breakout/ATtiny85_breakout.kicad_pcb (KiCad board)
At the start: 2 copper layers, 80.3 x 58.6 mm, 31 parts, among them J1 Conn_01x03_Female, J2 USB_B_Micro, J3 Conn_01x06_Female, J4 Conn_01x03_Female, U1 LM7805_TO220, U2 ATtiny85-20PU

Commit message: Añadimos modificaciones en el diseño
Parts:
- removed the REF** at (148.8, 41.5)
Other:
- board text added: "Piensa 3D 2019"
- board text removed: "Piensa 3D - 2019"
